File: Verstärker/Verstärker.kicad_pcb (KiCad board)
At the start: 2 copper layers, 99.5 x 53 mm, 63 parts, among them J3 ACJS-MHOM, J4 ACJS-MHOM, Q1 MJE182G, Q12 MMBT5401, Q12&Q13_E TP9, Q12_B TP4, Q12_C TP10, Q13 MMBT5401, Q13&Q12_C TP11, Q13_E TP8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

Commit message: do not include in position files bei testpoints
Parts:
- GND: value TP12 -> test_point
- GND: value H7 -> Mounting Hole with connection
- GND, GND4, GND5, GND6, GND7: value H5 -> Mounting Hole with connection
- IN: value H2 -> Mounting Hole with connection
- IN_AMP_B: value H9 -> Mounting Hole with connection
- Input: value TP5 -> test_point
- OUT: value H8 -> Mounting Hole with connection
- OUT_AMP_B: value H1 -> Mounting Hole with connection
- Out: value TP1 -> test_point
- Q12&Q13_E: value TP9 -> test_point
- Q12_B: value TP4 -> test_point
- Q12_C: value TP10 -> test_point
- Q13&Q12_C: value TP11 -> test_point
- Q13_E: value TP8 -> test_point
- Q1_E: value TP2 -> test_point
- Q2_E: value TP3 -> test_point
- Q3_C: value TP6 -> test_point
- Q3_E: value TP7 -> test_point
- VCC+: value H3 -> Mounting Hole with connection
- VCC-: value H4 -> Mounting Hole with connection
- VCC_GND: value H6 -> Mounting Hole with connection
Changed lines of the file:
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@@
 			)
 		)
-		(property "Value" "TP12"
+		(property "Value" "test_point"
 			(at 0 2.05 0)
 			(layer "F.Fab")
@@
 			)
 		)
-		(property "Description" "test point"
+		(property "Description" "TP12"
 			(at 0 0 0)
 			(unlocked yes)
@@
 		(sheetname "/")
 		(sheetfile "Verstärker.kicad_sch")
-		(attr exclude_from_pos_files)
+		(attr exclude_from_pos_files exclude_from_bom dnp)
 		(fp_circle
 			(center 0 0)
@@
 			)
 		)
-		(property "Value" "TP10"
+		(property "Value" "test_point"
 			(at 0 2.05 0)
 			(layer "F.Fab")
@@
 			)
 		)
-		(property "Description" "test point"
+		(property "Description" "TP10"
 			(at 0 0 0)
 			(unlocked yes)
@@
 		(sheetname "/")
 		(sheetfile "Verstärker.kicad_sch")
-		(attr exclude_from_pos_files)
+		(attr exclude_from_pos_files exclude_from_bom dnp)
 		(fp_circle
 			(center 0 0)
@@
 			)
 		)
-		(property "Value" "H9"
+		(property "Value" "Mounting Hole with connection"
 			(at 0 3.2 0)
 			(layer "F.Fab")
@@
 			)
 		)
-		(property "Description" "Mounting Hole with connection"
+		(property "Description" "H9"
 			(at 0 0 0)
 			(unlocked yes)
@@
 			)
 		)
-		(property "Value" "TP5"
+		(property "Value" "test_point"
 			(at 0 2.05 0)
 			(layer "F.Fab")
@@
 			)
 		)
-		(property "Description" "test point"
+		(property "Description" "TP5"
 			(at 0 0 0)
 			(unlocked yes)
@@
 		(sheetname "/")
 		(sheetfile "Verstärker.kicad_sch")
-		(attr exclude_from_pos_files)
+		(attr exclude_from_pos_files exclude_from_bom dnp)
 		(fp_circle
 			(center 0 0)
@@
 			)
 		)
-		(property "Value" "H7"
+		(property "Value" "Mounting Hole with connection"
 			(at 0 3.2 0)
 			(layer "F.Fab")
@@
 			)
 		)
-		(property "Description" "Mounting Hole with connection"
+		(property "Description" "H7"
 			(at 0 0 0)
 			(unlocked yes)
@@
 			)
 		)
-		(property "Value" "TP2"
+		(property "Value" "test_point"
 			(at 0 2.05 0)
 			(layer "F.Fab")
@@
 			)
 		)
-		(property "Description" "test point"
+		(property "Description" "TP2"
 			(at 0 0 0)
 			(unlocked yes)
@@
 		(sheetname "/")
 		(sheetfile "Verstärker.kicad_sch")
-		(attr exclude_from_pos_files)
+		(attr exclude_from_pos_files exclude_from_bom dnp)
 		(fp_circle
 			(center 0 0)
@@
 			)
 		)
-		(property "Value" "H1"
+		(property "Value" "Mounting Hole with connection"
 			(at 0 3.2 0)
 			(layer "F.Fab")
@@
 			)
 		)
-		(property "Description" "Mounting Hole with connection"
+		(property "Description" "H1"
 			(at 0 0 0)
 			(unlocked yes)
@@
 			)
 		)
-		(property "Value" "H6"
+		(property "Value" "Mounting Hole with connection"
 			(at 0 3.2 0)
 			(layer "F.Fab")
@@
 			)
 		)
-		(property "Description" "Mounting Hole with connection"
+		(property "Description" "H6"
 			(at 0 0 0)
 			(unlocked yes)
@@
 			)
 		)
-		(property "Value" "TP9"
+		(property "Value" "test_point"
 			(at 0 2.05 0)
 			(layer "F.Fab")
@@
 			)
 		)
-		(property "Description" "test point"
+		(property "Description" "TP9"
 			(at 0 0 0)
 			(unlocked yes)
@@
 		(sheetname "/")
 		(sheetfile "Verstärker.kicad_sch")
-		(attr exclude_from_pos_files)
+		(attr exclude_from_pos_files exclude_from_bom dnp)
 		(fp_circle
 			(center 0 0)
@@
 			)
 		)
-		(property "Value" "TP3"
+		(property "Value" "test_point"
 			(at 0 2.05 0)
 			(layer "F.Fab")
@@
 			)
 		)
-		(property "Description" "test point"
+		(property "Description" "TP3"
 			(at 0 0 0)
 			(unlocked yes)
@@
 			)
 		)
-		(property "Value" "H4"
+		(property "Value" "Mounting Hole with connection"
 			(at 0 3.2 0)
 			(layer "F.Fab")
@@
 			)
 		)
-		(property "Description" "Mounting Hole with connection"
+		(property "Description" "H4"
 			(at 0 0 0)
 			(unlocked yes)
@@
 			)
 		)
-		(property "Value" "H5"
+		(property "Value" "Mounting Hole with connection"
 			(at 0 3.2 0)
 			(layer "F.Fab")
@@
 			)
 		)
-		(property "Description" "Mounting Hole with connection"
+		(property "Description" "H5"
 			(at 0 0 0)
 			(unlocked yes)
@@
 			)
 		)
-		(property "Value" "H3"
+		(property "Value" "Mounting Hole with connection"
 			(at 0 3.2 0)
 			(layer "F.Fab")
@@
 			)
 		)
-		(property "Description" "Mounting Hole with connection"
+		(property "Description" "H3"
 			(at 0 0 0)
 			(unlocked yes)
@@
 			)
 		)
-		(property "Value" "H5"
+		(property "Value" "Mounting Hole with connection"
 			(at 0 3.2 0)
 			(layer "F.Fab")
@@
 			)
 		)
-		(property "Description" "Mounting Hole with connection"
+		(property "Description" "H5"
 			(at 0 0 0)
 			(unlocked yes)
@@
 			)
 		)
-		(property "Value" "TP8"
+		(property "Value" "test_point"
 			(at 0 2.05 0)
 			(layer "F.Fab")
@@
 			)
 		)
-		(property "Description" "test point"
+		(property "Description" "TP8"
 			(at 0 0 0)
 			(unlocked yes)
@@
 		(sheetname "/")
 		(sheetfile "Verstärker.kicad_sch")
-		(attr exclude_from_pos_files)
+		(attr exclude_from_pos_files exclude_from_bom dnp)
 		(fp_circle
 			(center 0 0)
@@
 			)
 		)
-		(property "Value" "H5"
+		(property "Value" "Mounting Hole with connection"
 			(at 0 3.2 0)
 			(layer "F.Fab")
@@
 			)
 		)
-		(property "Description" "Mounting Hole with connection"
+		(property "Description" "H5"
 			(at 0 0 0)
 			(unlocked yes)
@@
 			)
 		)
-		(property "Value" "TP6"
+		(property "Value" "test_point"
 			(at 0 2.05 0)
 			(layer "F.Fab")
@@
 			)
 		)
-		(property "Description" "test point"
+		(property "Description" "TP6"
 			(at 0 0 0)
 			(unlocked yes)
@@
 		(sheetname "/")
 		(sheetfile "Verstärker.kicad_sch")
-		(attr exclude_from_pos_files)
+		(attr exclude_from_pos_files exclude_from_bom dnp)
 		(fp_circle
 			(center 0 0)
@@
 			)
 		)
-		(property "Value" "TP4"
+		(property "Value" "test_point"
 			(at 0 2.05 0)
 			(layer "F.Fab")
@@
 			)
 		)
-		(property "Description" "test point"
+		(property "Description" "TP4"
 			(at 0 0 0)
 			(unlocked yes)
@@
 		(sheetname "/")
 		(sheetfile "Verstärker.kicad_sch")
-		(attr exclude_from_pos_files)
+		(attr exclude_from_pos_files exclude_from_bom dnp)
 		(fp_circle
 			(center 0 0)
@@
 			)
 		)
-		(property "Value" "TP11"
+		(property "Value" "test_point"
 			(at 0 2.05 0)
 			(layer "F.Fab")
@@
 			)
 		)
-		(property "Description" "test point"
+		(property "Description" "TP11"
 			(at 0 0 0)
 			(unlocked yes)
@@
 		(sheetname "/")
 		(sheetfile "Verstärker.kicad_sch")
-		(attr exclude_from_pos_files)
+		(attr exclude_from_pos_files exclude_from_bom dnp)
 		(fp_circle
 			(center 0 0)
@@
 			)
 		)
-		(property "Value" "H5"
+		(property "Value" "Mounting Hole with connection"
 			(at 0 3.2 0)
 			(layer "F.Fab")
@@
 			)
 		)
-		(property "Description" "Mounting Hole with connection"
+		(property "Description" "H5"
 			(at 0 0 0)
 			(unlocked yes)
@@
 			)
 		)
-		(property "Value" "H5"
+		(property "Value" "Mounting Hole with connection"
 			(at 0 3.2 0)
 			(layer "F.Fab")
@@
 			)
 		)
-		(property "Description" "Mounting Hole with connection"
+		(property "Description" "H5"
 			(at 0 0 0)
 			(unlocked yes)
@@
 			)
 		)
-		(property "Value" "H8"
+		(property "Value" "Mounting Hole with connection"
 			(at 0 3.2 0)
 			(layer "F.Fab")
@@
 			)
 		)
-		(property "Description" "Mounting Hole with connection"
+		(property "Description" "H8"
 			(at 0 0 0)
 			(unlocked yes)
@@
 			)
 		)
-		(property "Value" "H2"
+		(property "Value" "Mounting Hole with connection"
 			(at 0 3.2 0)
 			(layer "F.Fab")
@@
 			)
 		)
-		(property "Description" "Mounting Hole with connection"
+		(property "Description" "H2"
 			(at 0 0 0)
 			(unlocked yes)
@@
 			)
 		)
-		(property "Value" "TP7"
+		(property "Value" "test_point"
 			(at 0 2.05 0)
 			(layer "F.Fab")
@@
 			)
 		)
-		(property "Description" "test point"
+		(property "Description" "TP7"
 			(at 0 0 0)
 			(unlocked yes)
@@
 		(sheetname "/")
 		(sheetfile "Verstärker.kicad_sch")
-		(attr exclude_from_pos_files)
+		(attr exclude_from_pos_files exclude_from_bom dnp)
 		(fp_circle
 			(center 0 0)
@@
 			)
 		)
-		(property "Value" "TP1"
+		(property "Value" "test_point"
 			(at 0 2.05 0)
 			(layer "F.Fab")
@@
 			)
 		)
-		(property "Description" "test point"
+		(property "Description" "TP1"
 			(at 0 0 0)
 			(unlocked yes)
@@
 		(sheetname "/")
 		(sheetfile "Verstärker.kicad_sch")
-		(attr exclude_from_pos_files)
+		(attr exclude_from_pos_files exclude_from_bom dnp)
 		(fp_circle
 			(center 0 0)
